File: Hardware/H7FC/CM4/H7MCU.kicad_sch (KiCad schematic)
At the start: 64 parts, among them IC2 STM32H747IIT6, J14 SWDIO, J15 Micro_SD_Card, Y1 16MHz

Commit message: Set initial cUbeMX Cconfig. Fixed Clock and GPIO bug
Parts:
- removed C18, C20, C21, C22, C23, C24, C48: 100n, Capacitor_SMD:C_0402_1005Metric, symbol Device:C_Small
- removed C44: 1u_X5R_0603, Capacitor_SMD:C_0603_1608Metric, symbol Device:C_Small
- removed C47: 4.7u, Capacitor_Tantalum_SMD:CP_EIA-3216-18_Kemet-A, symbol Device:C_Polarized_Small
- removed C49: 2.2u, Capacitor_SMD:C_0603_1608Metric, symbol Device:C_Small
- removed IC2: STM32H747IIT6, QFP50P2600X2600X160-176N, symbol SamacSys_Parts:STM32H747IIT6
- removed R14: 10k, Resistor_SMD:R_0402_1005Metric, symbol Device:R_Small
- added R6: 10k, Resistor_SMD:R_0402_1005Metric, symbol Device:R_Small
- C16: value 100n -> 1u
- C17: value 100n -> 1u_X5R_0603; footprint Capacitor_SMD:C_0402_1005Metric -> Capacitor_SMD:C_0603_1608Metric; Digi-Key_PN 587-1226-2-ND -> (none); LCSC Part # C1525 -> C15849; Seeed SKU 302010024 -> 302010139
- IC2: renamed from IC?; footprint QFP50P2200X2200X160-144N -> SamacSys_Parts:QFP50P2200X2200X160-144N
- S1: footprint TL1105CF160Q -> SamacSys_Parts:TL1105CF160Q
- S2: footprint SOT175P420X230-3N -> SamacSys_Parts:SOT175P420X230-3N
Connections:
- net VCAP1 is gone; now on net VCAP: C45.1, C46.1
- net +3.3VA: now also IC2.36 (VDDA)
- net ANALOG_IN: now also IC2.52 (PF11)
- net BOOT0: now also IC2.135 (BOOT0)
- net GND: now also IC2.104 (VSS_10), IC2.118 (VSS_11), IC2.12 (VSS_2), IC2.128 (VSS_12), IC2.14 (VSSSMPS), IC2.141 (VSS_13), IC2.16 (VDDSMPS), IC2.17 (VFBSMPS), IC2.18 (VSS_3), IC2.33 (VSS_4), IC2.34 (VSSA), IC2.41 (VSS_5), IC2.55 (VSS_6), IC2.6 (VSS_1), IC2.69 (VSS_7), IC2.80 (VSS_8), IC2.89 (VSS_9)
- net HSE_IN: now also IC2.25 (PH0-OSC_IN)
- net HSE_OUT: now also IC2.26 (PH1-OSC_OUT)
- net I2C1_SCL: now also IC2.136 (PB8)
- net I2C1_SDA: now also IC2.137 (PB9)
- net I2C2_SCL: now also IC2.66 (PB10)
- net I2C2_SDA: now also IC2.67 (PB11)
- net LED_A: now also IC2.57 (PE7)
- net LED_B: now also IC2.58 (PE8)
- net LED_C: now also IC2.22 (PF8)
- net LED_D: now also IC2.23 (PF9)
- net LSM9DS1_CS_AG: now also IC2.2 (PE3)
- net LSM9DS1_CS_M: now also IC2.131 (PB4)
- net LSM9DS1_DEN_AG: now also IC2.123 (PG10)
- net LSM9DS1_DRDY_M: now also IC2.127 (PG14)
- net LSM9DS1_INT1_AG: now also IC2.125 (PG12)
- net LSM9DS1_INT2_AG: now also IC2.124 (PG11)
- net LSM9DS1_INT_M: now also IC2.126 (PG13)
- net LSM9DS1_SDO_AG: now also IC2.3 (PE4)
- net LSM9DS1_SDO_M: now also IC2.1 (PE2)
- net M8Q_NRST: now also IC2.85 (PD15)
- net M8Q_PPS: now also IC2.84 (PD14)
- net M8Q_RX: now also IC2.76 (PD8)
- net M8Q_TX: now also IC2.77 (PD9)
- net NRST: now also IC2.27 (NRST)
- net SBUS_RX: now also IC2.38 (PA1)
- net SDMMC_CK: now also IC2.111 (PC12)
- net SDMMC_CMD: now also IC2.114 (PD2)
- net SDMMC_D0: now also IC2.95 (PC8)
- net SDMMC_D1: now also IC2.96 (PC9)
- net SDMMC_D2: now also IC2.109 (PC10)
- net SDMMC_D3: now also IC2.110 (PC11)
- net SPI1_MISO: now also IC2.45 (PA6)
- net SPI1_MOSI: now also IC2.46 (PA7)
- net SPI1_NCS: now also IC2.43 (PA4)
- net SPI1_SCK: now also IC2.44 (PA5)
- net SWCLK: now also IC2.107 (PA14)
- net SWDIO: now also IC2.102 (PA13)
- net SWO: now also IC2.130 (PB3)
- net TIM1_CH1: now also IC2.97 (PA8)
- net TIM1_CH2: now also IC2.61 (PE11)
- net TIM1_CH3: now also IC2.63 (PE13)
- net TIM1_CH4: now also IC2.64 (PE14)
- net UART7_RX: now also IC2.20 (PF6)
- net UART7_TX: now also IC2.21 (PF7)
- net USB_D_N: now also IC2.100 (PA11)
- net USB_D_P: now also IC2.101 (PA12)
- net VREF+: now also IC2.35 (VREF+)
- net VCAP: now reaches IC2.103 (VCAP_2)
- net VCAP: now also IC2.140 (VCAP_3), IC2.68 (VCAP_1)
- net VDDLDO: now reaches IC2.105 (VDDLDO_2)
- net VDDLDO: now also C15.1, C17.1, C19.1, C29.1, C30.1, C31.1, C32.1, C33.1, C34.1, C35.1, C36.1, C37.1, C38.1, C39.1, C40.1, FB2.1, IC2.106 (VDD_10), IC2.119 (VDD_11), IC2.129 (VDD_12), IC2.13 (VDD_2), IC2.143 (VDDLDO_3), IC2.144 (VDD_13), IC2.19 (VDD_3), IC2.32 (VDD_4), IC2.42 (VDD_5), IC2.56 (VDD_6), IC2.7 (VDD_1), IC2.70 (VDDLDO_1), IC2.71 (VDD_7), IC2.79 (VDD_8), IC2.90 (VDD50USB), IC2.91 (VDD33USB), IC2.92 (VDD_9), J14.1 (Pin_1), J15.4 (VDD), R15.1, R16.2, R17.1, R18.2, R27.2, R28.2, R29.2, R30.2, R31.2, S2.1, R6.1
- net at IC2.142 (PDR_ON): now also R6.2
- net VBAT: now reaches IC2.8 (VBAT)
- net VBAT: now also C16.1
- removed net +3.3VG: C15.1, C16.1, C17.1, C19.1, C29.1, C30.1, C31.1, C32.1, C33.1, C34.1, C35.1, C36.1, C37.1, C38.1, C39.1, C40.1, FB2.1, J14.1 (Pin_1), J15.4 (VDD), R15.1, R16.2, R17.1, R18.2, R27.2, R28.2, R29.2, R30.2, R31.2, S2.1
- no-connect marks 74 -> 56
Other:
- moved on the sheet: C15, C19, C29, C30, C31, C32, C33, C34, C35, C36, C37, C38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
