File: Hardware/H7FC/CM4/power.kicad_sch (KiCad schematic)
At the start: 18 parts, among them IC1 ADP7156ARDZ-3.3-R7, J2 USB_C_Receptacle_USB2.0, J3 Conn_01x02, Q1 AO3401A

Commit message: Set initial cUbeMX Cconfig. Fixed Clock and GPIO bug
Parts:
- removed D2: SS14, Diode_SMD:D_SMA, symbol pspice:DIODE
- removed J3: Conn_01x02, Connector_Molex:Molex_PicoBlade_53261-0271_1x02-1MP_P1.25mm_Horizontal, symbol Connector_Generic:Conn_01x02
- removed JP1: Jumper_3_Open, Jumper:SolderJumper-3_P1.3mm_Open_RoundedPad1.0x1.5mm, symbol Jumper:Jumper_3_Open
- FB1: footprint Inductor_SMD:L_0805_2012Metric -> Inductor_SMD:L_0603_1608Metric
- gave numbers to parts that had none: 2
Connections:
- net USB_D+: now also U4.6 (I/O1); no longer U4.4 (I/O2)
- net USB_D-: now also U4.4 (I/O2); no longer U4.6 (I/O1)
- net USB_D_P: now reaches U4.1 (I/O1)
- net USB_D_N: now reaches U4.3 (I/O2)
Other:
- moved on the sheet: D1, R1, U4
