File: Hardware/CM4 Version/H7MCU.kicad_sch (KiCad schematic)
At the start: 73 parts, among them IC2 STM32H747IIT6, J13 USB_B_Micro, J14 SWDIO, J15 Micro_SD_Card, U4 USBLC6-2SC6, Y1 16MHz

Commit message: Remove CM4-Backups
Parts:
- removed C15, C47: 4.7u, Capacitor_Tantalum_SMD:CP_EIA-3216-18_Kemet-A, symbol Device:C_Polarized_Small
- removed C16, C17, C19, C33, C48, C52: 100n, Capacitor_SMD:C_0402_1005Metric, symbol Device:C_Small
- removed C25, C27: 1u, Capacitor_Tantalum_SMD:CP_EIA-3216-18_Kemet-A, symbol Device:C_Polarized_Small
- removed C41, C43: 10u, Capacitor_SMD:C_0603_1608Metric, symbol Device:C_Small
- removed C42: 220p, Capacitor_SMD:C_0402_1005Metric, symbol Device:C_Small
- removed C44: 1u_X5R_0603, Capacitor_SMD:C_0603_1608Metric, symbol Device:C_Small
- removed C45, C46: 4.7u, Capacitor_SMD:C_0603_1608Metric, symbol Device:C_Small
- removed C49: 2.2u, Capacitor_SMD:C_0603_1608Metric, symbol Device:C_Small
- removed C50, C51: 12p, Capacitor_SMD:C_0402_1005Metric, symbol Device:C_Small
- removed D3: SD103AWS-TP, SamacSys_Parts:SOD2512X115N, symbol SamacSys_Parts:SD103AWS-TP
- removed D7: LED_Red, LED_SMD:LED_0603_1608Metric, symbol Device:LED_Small
- removed FB3: 100 @100Mhz, Inductor_SMD:L_0603_1608Metric, symbol Device:FerriteBead_Small
- removed FB4: 18 @100Mhz, Inductor_SMD:L_0603_1608Metric, symbol Device:FerriteBead_Small
- removed IC2: STM32H747IIT6, SamacSys_Parts:QFP50P2600X2600X160-176N, symbol SamacSys_Parts:STM32H747IIT6
- removed J13: USB_B_Micro, Connector_USB:USB_Micro-B_Molex-105017-0001, symbol Connector:USB_B_Micro
- removed L3: 2.2uH, Inductor_SMD:L_0805_2012Metric, symbol Device:L_Small
- removed R23, R24, R25: 2k2, Resistor_SMD:R_0603_1608Metric, symbol Device:R_Small
- removed R26: 47, Resistor_SMD:R_0402_1005Metric, symbol Device:R_Small
- removed R28, R29, R30, R31: 47k, Resistor_SMD:R_0402_1005Metric, symbol Device:R_Small_US
- removed R32: 10k, Resistor_SMD:R_0402_1005Metric, symbol Device:R_Small
- removed S1: TL1105CF160Q, SamacSys_Parts:TL1105CF160Q, symbol SamacSys_Parts:TL1105CF160Q
- removed S2: TDD01H0SB1R, SamacSys_Parts:SOT175P420X230-3N, symbol SamacSys_Parts:TDD01H0SB1R
- removed U4: USBLC6-2SC6, Package_TO_SOT_SMD:SOT-23-6, symbol Power_Protection:USBLC6-2SC6
- added C17, C33: 1u, Capacitor_Tantalum_SMD:CP_EIA-3216-18_Kemet-A, symbol Device:C_Polarized_Small
- added C19: 4.7u, Capacitor_Tantalum_SMD:CP_EIA-3216-18_Kemet-A, symbol Device:C_Polarized_Small
- added C25, C27: 100n, Capacitor_SMD:C_0402_1005Metric, symbol Device:C_Small
- added D3: LED_Red, LED_SMD:LED_0603_1608Metric, symbol Device:LED_Small
- added IC2: STM32H745ZIT6, SamacSys_Parts:QFP50P2200X2200X160-144N, symbol SamacSys_Parts:STM32H745ZIT6
- added R12, R28: 10k, Resistor_SMD:R_0402_1005Metric, symbol Device:R_Small
- added R19, R20: 2k2, Resistor_SMD:R_0603_1608Metric, symbol Device:R_Small
- added R23, R24, R25, R26: 47k, Resistor_SMD:R_0402_1005Metric, symbol Device:R_Small_US
- added S1: TDD01H0SB1R, SamacSys_Parts:SOT175P420X230-3N, symbol SamacSys_Parts:TDD01H0SB1R
- C35, C37: value 100n -> 2.2u; footprint Capacitor_SMD:C_0402_1005Metric -> Capacitor_SMD:C_0603_1608Metric; Digi-Key_PN 587-1226-2-ND -> (none); LCSC Part # C1525 -> C19666; Seeed SKU 302010024 -> 302010111
- C36: value 100n -> 1u
- C38: value 100n -> 1u_X5R_0603; footprint Capacitor_SMD:C_0402_1005Metric -> Capacitor_SMD:C_0603_1608Metric; Digi-Key_PN 587-1226-2-ND -> (none); LCSC Part # C1525 -> C15849; Seeed SKU 302010024 -> 302010139
- C39, C40: value 100n -> 12p; Digi-Key_PN 587-1226-2-ND -> (none); LCSC Part # C1525 -> C1547; Seeed SKU 302010024 -> 302010049
- D4, D5, D6: LCSC Part # (none) -> C72043; Seeed SKU 304090042 -> (none)
- FB2: Digi-Key_PN 445-1564-2-ND -> (none)
- J15: Digi-Key_PN HR1964TR-ND -> (none)
- R13: LCSC Part # (none) -> C23182
- R14: value 10k -> 4k7; Digi-Key_PN RG10P10.0KDTR-ND -> (none); LCSC Part # C25744 -> C23162; Seeed SKU 301010004 -> 301010010
- R15, R16, R17: LCSC Part # (none) -> C23162
- R18: value 4k7 -> 2k2; footprint Resistor_SMD:R_0402_1005Metric -> Resistor_SMD:R_0603_1608Metric; LCSC Part # (none) -> C4190; Seeed SKU 301010010 -> 301010039
- R21: value 560 -> 2k2; footprint Resistor_SMD:R_0402_1005Metric -> Resistor_SMD:R_0603_1608Metric; Digi-Key_PN 311-560GRTR-ND -> (none); Digikey Link https://www.digikey.co.uk/en/products/detail/yageo/RC0603JR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 -> (none); LCSC Part # (none) -> C4190; Manufacturer_Part_Number RC0603JR-07560RL -> (none); Seeed SKU (none) -> 301010039
- R22: value 2k2 -> 47; footprint Resistor_SMD:R_0603_1608Metric -> Resistor_SMD:R_0402_1005Metric; LCSC Part # (none) -> C23182; Seeed SKU 301010039 -> 301010878
- R27: LCSC Part # C25792 -> C25792
- Y1: LCSC Part # (none) -> C13738
Connections:
- net USB_OTG_ID is gone; now on net GND: R21.2
- net +3.3VA: now also C34.2, C33.1, IC2.36 (VDDA); no longer C28.2
- net ANALOG_IN: now also IC2.52 (PF11)
- net BOOT0: now also IC2.135 (BOOT0), R28.2
- net GND: now also C18.1, C26.2, C28.2, C34.1, C39.1, R18.2, C17.2, C19.2, C25.2, C27.2, C33.2, IC2.104 (VSS_10), IC2.118 (VSS_11), IC2.12 (VSS_2), IC2.128 (VSS_12), IC2.14 (VSSSMPS), IC2.141 (VSS_13), IC2.16 (VDDSMPS), IC2.17 (VFBSMPS), IC2.18 (VSS_3), IC2.33 (VSS_4), IC2.34 (VSSA), IC2.41 (VSS_5), IC2.55 (VSS_6), IC2.6 (VSS_1), IC2.69 (VSS_7), IC2.80 (VSS_8), IC2.89 (VSS_9), R19.2, R20.2, S1.2; no longer C18.2, C26.1, C28.1, C34.2, C39.2, R22.2
- net HSE_IN: now also C40.1, IC2.25 (PH0-OSC_IN)
- net HSE_OUT: now also R22.1, IC2.26 (PH1-OSC_OUT)
- net I2C1_SCL: now also R14.2, IC2.136 (PB8); no longer R15.2
- net I2C1_SDA: now also R15.1, IC2.137 (PB9); no longer R16.1
- net I2C2_SCL: now also R17.1, IC2.66 (PB10); no longer R18.1
- net I2C2_SDA: now also R16.2, IC2.67 (PB11); no longer R17.2
- net LED_A: now also D5.2 (A), IC2.57 (PE7); no longer D6.2 (A)
- net LED_B: now also D3.2 (A), IC2.58 (PE8); no longer D4.2 (A)
- net LED_C: now also D6.2 (A), IC2.22 (PF8)
- net LED_D: now also D4.2 (A), IC2.23 (PF9); no longer D5.2 (A)
- net LSM9DS1_CS_AG: now also IC2.2 (PE3)
- net LSM9DS1_CS_M: now also IC2.131 (PB4)
- net LSM9DS1_DEN_AG: now also IC2.123 (PG10)
- net LSM9DS1_DRDY_M: now also IC2.127 (PG14)
- net LSM9DS1_INT1_AG: now also IC2.125 (PG12)
- net LSM9DS1_INT2_AG: now also IC2.124 (PG11)
- net LSM9DS1_INT_M: now also IC2.126 (PG13)
- net LSM9DS1_SDO_AG: now also IC2.3 (PE4)
- net LSM9DS1_SDO_M: now also IC2.1 (PE2)
- net M8Q_NRST: now also IC2.85 (PD15)
- net M8Q_PPS: now also IC2.84 (PD14)
- net M8Q_RX: now also IC2.76 (PD8)
- net M8Q_TX: now also IC2.77 (PD9)
- net NRST: now also IC2.27 (NRST)
- net SBUS_RX: now also IC2.38 (PA1)
- net SDMMC_CK: now also IC2.111 (PC12)
- net SDMMC_CMD: now also IC2.114 (PD2), R25.1
- net SDMMC_D0: now also IC2.95 (PC8), R26.1
- net SDMMC_D1: now also R27.1, IC2.96 (PC9)
- net SDMMC_D2: now also IC2.109 (PC10), R23.1; no longer R27.1
- net SDMMC_D3: now also IC2.110 (PC11), R24.1
- net SPI1_MISO: now also IC2.45 (PA6)
- net SPI1_MOSI: now also IC2.46 (PA7)
- net SPI1_NCS: now also IC2.43 (PA4)
- net SPI1_SCK: now also IC2.44 (PA5)
- net SWCLK: now also IC2.107 (PA14)
- net SWDIO: now also IC2.102 (PA13)
- net SWO: now also IC2.130 (PB3)
- net TIM1_CH1: now also IC2.97 (PA8)
- net TIM1_CH2: now also IC2.61 (PE11)
- net TIM1_CH3: now also IC2.63 (PE13)
- net TIM1_CH4: now also IC2.64 (PE14)
- net UART7_RX: now also IC2.20 (PF6)
- net UART7_TX: now also IC2.21 (PF7)
- net USB_D_N: now also IC2.100 (PA11)
- net USB_D_P: now also IC2.101 (PA12)
- net VREF+: now also C18.2, C17.1, IC2.35 (VREF+); no longer C26.2
- net at D5.1 (K): now also R20.1
- net at D4.1 (K): now also R19.1; no longer R22.1
- net at D6.1 (K): now also R21.1
- net at Y1.3: now also C39.2, R22.2
- net +3.3VG renamed VDDLDO
- net VDDLDO: now also C26.1, C28.1, R15.2, R16.1, R17.2, C19.1, C25.1, C27.1, IC2.105 (VDDLDO_2), IC2.106 (VDD_10), IC2.119 (VDD_11), IC2.129 (VDD_12), IC2.13 (VDD_2), IC2.143 (VDDLDO_3), IC2.144 (VDD_13), IC2.19 (VDD_3), IC2.32 (VDD_4), IC2.42 (VDD_5), IC2.56 (VDD_6), IC2.7 (VDD_1), IC2.70 (VDDLDO_1), IC2.71 (VDD_7), IC2.79 (VDD_8), IC2.90 (VDD50USB), IC2.91 (VDD33USB), IC2.92 (VDD_9), R12.1, R23.2, R24.2, R25.2, R26.2, S1.1; no longer C18.1, C34.1, C35.1, C36.1, C37.1, C39.1, C40.1, R15.1, R16.2, R17.1, R18.2
- new net: D3.1 (K), R18.1
- new net: R28.1, S1.3 (C)
- new net: IC2.142 (PDR_ON), R12.2
- new net VBAT: C36.1, IC2.8 (VBAT)
- new net VCAP: C35.1, C37.1, IC2.103 (VCAP_2), IC2.140 (VCAP_3), IC2.68 (VCAP_1)
- no-connect marks 70 -> 56
Other:
- note removed: "Do you need an EMI filter? emif06-hsd03f3"
- note removed: "Place near 2.2uH"
- note removed: "RESET BUTTON"
- note removed: "SMPS CIRCUITRY"
