File: Hardware/CM4 Version/cm4-high-speed.kicad_sch (KiCad schematic)
At the start: 1 part

Commit message: Remove CM4-Backups
Parts:
- Module1: Digikey Link https://www.digikey.co.uk/en/products/detail/hirose-electri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 -> (none); Seeed SKU 320210381 -> (none)
